Commit message: working gazebo fortress sim

File: NAV/rover_workspace/src/roverrobotics_ros2/roverrobotics_description/urdf/accessories/rplidar_s2.urdf (robot description, URDF)
Before this commit: robot rplidar_s2, 1 links, 1 joints
Links:
- link lidar_link: mass None -> 0.19; geometry collision cylinder length=0.04 radius=0.04; visual mesh filename=file://$(find roverrobotics_description)/meshes/rplidar_s2.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
Joints:
- joint lidar_to_payload: origin xyz=0.174 0 0.145 rpy=0 0 3.1415 -> xyz=0.174 0 0.2 rpy=0 0 3.1415
